File: keyscar_kicad/keyscar_kicad.kicad_pcb (KiCad board)
At the start: 2 copper layers, 21 x 26.8 mm, 31 parts, among them SW1 SSSS211603, SW2 SSSS211603, SW5_MASTER_EXEC1 TSA453G50-250, SW6_SLAVE_EXEC2 TSA453G50-250

Commit message: safety commit again
Parts:
- SW_CHIP_RST3, SW_MASTER_BOOT1, SW_SLAVE_BOOT2: value EVQP2D02Q -> EVQP2202M; footprint Library:KEY-SMD_4P-L4.7-W3.5-P1.70-LS5.5 -> Library:SW-SMD_L4.7-W3.5-P2.00-LS5.2_EVQP2202M
- USBC_MALE1: value 918-118A2021S40003 -> 918-118A2021Y40005; footprint Library:USB-C-SMD_918-118A2021S40003 -> Library:USB-C-SMD_918-118A2021Y40005
- moved USBC_MALE1 0.88 mm to (255.7, 73.6)
- moved SW_MASTER_BOOT1 0.11 mm to (257.9, 80.1), turned to 0 degrees
- moved SW_SLAVE_BOOT2 0.10 mm to (258.0, 88.0), turned to 180 degrees
- moved SW_CHIP_RST3 0.05 mm to (248.1, 86.8), turned to 0 degrees
Connections:
- USBC_MALE1 pad B12: GND -> unconnected-(USBC_MALE1-GND-PadB12)
Routing:
- net USB C VBUS: track 10.9 -> 21.9 mm, vias 1 -> 2
- net GND: track 123.7 -> 116.8 mm, vias 13 -> 16
- net MASTERC D-: track 7.47 -> 10.8 mm
- net Net-(USBC_MALE1-CC2): track 8.63 -> 6.35 mm, vias 1 -> 2
- net Net-(USBC_MALE1-CC1): track 1.33 -> 3.36 mm
- net MASTERC D+: track 11.7 -> 10.3 mm, vias 3 -> 2

Commit message: :( Old peak 2 sided
Other:
- board size 21 x 26.8 mm -> 21 x 27.3 mm
